File: KiCad/nucleo_shield.kicad_pcb (KiCad board)
At the start: 2 copper layers, 55.4 x 51.2 mm, 33 parts, among them J13 Conn_01x10_2,54mm, J4 Conn_01x08_2,54mm, J5 Conn_01x06_2,54mm, J7 Conn_01x08_2,54mm, J8 DC_Jack_2.5mm, U1 ADA4625-2ARDZ, U3 OPA197xD, U4 LD1117S50TR_SOT223

Commit message: added 12v source for nucleo
Parts:
- renumbered POL3 to POL2, POL2 to POL3
Connections:
- J4 pad 7: unconnected-(J4-Pin_7-Pad7) -> GND
- J4 pad 8: unconnected-(J4-Pin_8-Pad8) -> 12V
Routing:
- net 12V: track 67.3 -> 122.5 mm
